File: I2CPANEL.brd (EAGLE design)
At the start: 100 x 30 mm, 26 parts, among them IC1 MCP23017SO, J1 M10-SOCKET, J2 I2C, J3 I2C

Commit message: Changed to I2C-BREAKOUT header for v3.0 release
Parts:
- removed J3: I2C, SuperHouse-Connectors:1X06-P
- added J4: M01-PLAIN, SuperHouse-Connectors:1X01
- added J6: I2C-BREAKOUT, SuperHouse-Connectors:2X03-SHROUDED
- J2: value I2C -> I2C-BREAKOUT; device SuperHouse-Connectors:1X06-P -> SuperHouse-Connectors:2X03-SHROUDED
- moved J2 23.8 mm to (21.0, 25.0), turned to 90 degrees
Connections:
- new net !RESET: IC1.18, J2.6, J6.6
- net !INT: now also J4.1; no longer J2.6, J3.6
- net GND: now also J6.4; no longer J3.4
- net SCL: now also J2.1, J6.1; no longer J2.2, J3.2
- net SDA: now also J2.2, J6.2; no longer J2.1, J3.1
- net VCC: now also J2.5, J6.5; no longer IC1.18, J2.3, J3.3
- net VIN: now also J2.3, J6.3; no longer J2.5, J3.5
Routing:
- net SDA: track 71.6 -> 140.4 mm
- net SCL: track 73.2 -> 131.6 mm
- net !RESET: track 0.00 -> 53.1 mm, vias 0 -> 1
- net !INT: track 50.2 -> 3.44 mm, vias 1 -> 0
- net VIN: track 2.54 -> 23.3 mm
- net GND: track 24.2 -> 31.7 mm
- net GPA6: track 51.5 -> 53.6 mm
Other:
- board text added: "!RST"
- board text added: "Copyright 2019-2020 SuperHouse Automation Pty Ltd Released under the TAPR Open Hardware License www.tapr.org/OHL"
- board text added: "I2C-BREAKOUT"
- board text added: "v3.0"
- board text removed: "Copyright 2019 SuperHouse Automation Pty Ltd Released under the TAPR Open Hardware License www.tapr.org/OHL"
- board text removed: "LED2"
- board text removed: "v2.0"
